File: line-interface/line-interface.kicad_pcb (KiCad board)
At the start: 2 copper layers, 0 parts

Commit message: Initial PCB component placement, start routing
Parts:
- added C1: 1u, Capacitors_SMD:C_0603, F.Cu at (127.0, 125.5)
- added C2: 1u, Capacitors_SMD:C_1210_HandSoldering, F.Cu at (175.0, 117.0)
- added C3: CP1, Capacitors_ThroughHole:CP_Radial_D8.0mm_P3.50mm, F.Cu at (157.0, 105.0)
- added C4: 1u, Capacitors_SMD:C_0603, F.Cu at (127.0, 127.0)
- added C5: 1u, Capacitors_SMD:C_1210_HandSoldering, F.Cu at (147.0, 102.0)
- added C6: 18p, Capacitors_SMD:C_0603, F.Cu at (116.8, 139.0)
- added C7: 1u, Capacitors_SMD:C_0603, F.Cu at (142.0, 114.8)
- added C8: 18p, Capacitors_SMD:C_0603, F.Cu at (117.0, 125.0)
- added C9: 1u, Capacitors_SMD:C_0603, F.Cu at (143.5, 131.0)
- added D1: D_TVS_ALT, Diodes_SMD:Diode-SMC_Handsoldering, F.Cu at (172.0, 125.0)
- added D2: 60V, Diodes_SMD:D_SMB_Handsoldering, F.Cu at (174.0, 113.0)
- added D3: 15V, Diodes_SMD:SOD-123, F.Cu at (163.0, 115.0)
- added D4: GREEN, LEDs:LED_0603, F.Cu at (129.2, 144.1)
- added D5: RED, LEDs:LED_0603, F.Cu at (131.8, 144.1)
- added D6: GREEN, LEDs:LED_0603, F.Cu at (140.0, 109.0)
- added IC1: ATTINY441-SSU, Housings_SOIC:SOIC-14_3.9x8.7mm_Pitch1.27mm, F.Cu at (130.0, 134.0)
- added J1: CONN_01X06, Pin_Headers:Pin_Header_Straight_1x06_Pitch2.54mm, F.Cu at (101.3, 117.0)
- added MK1: Mounting_Hole, Mounting_Holes:MountingHole_3.2mm_M3, F.Cu at (176.0, 145.0)
- added MK2: Mounting_Hole, Mounting_Holes:MountingHole_3.2mm_M3, F.Cu at (104.0, 104.0)
- added MK3: Mounting_Hole, Mounting_Holes:MountingHole_3.2mm_M3, F.Cu at (104.0, 145.0)
- added MK4: Mounting_Hole, Mounting_Holes:MountingHole_3.2mm_M3, F.Cu at (176.0, 104.0)
- added P1: CONN_02X03, Pin_Headers:Pin_Header_Straight_2x03_Pitch2.54mm, F.Cu at (134.0, 121.0)
- added P2: CONN_01X04, Pin_Headers:Pin_Header_Straight_1x04_Pitch2.54mm, F.Cu at (177.1, 130.0)
- added Q1: NDT2955, TO_SOT_Packages_SMD:TO-252-2Lead, F.Cu at (163.7, 108.3)
- added R1: 10, Resistors_SMD:R_0805_HandSoldering, F.Cu at (176.3, 120.0)
- added R2: 10k, Resistors_SMD:R_0603, F.Cu at (166.8, 115.0)
- added R3: 10k, Resistors_SMD:R_0603, F.Cu at (129.2, 141.2)
- added R4: 10k, Resistors_SMD:R_0603, F.Cu at (126.8, 128.5)
- added R5: 18.2k, Resistors_SMD:R_0603_HandSoldering, F.Cu at (142.0, 107.0)
- added R6: 10k, Resistors_SMD:R_0603, F.Cu at (131.8, 141.0)
- added R7: 6.04k, Resistors_SMD:R_0603_HandSoldering, F.Cu at (142.0, 111.1)
- added R8: 330, Resistors_SMD:R_0603, F.Cu at (140.0, 112.0)
- added U1: LR12K, TO_SOT_Packages_SMD:TO-252-2Lead, F.Cu at (147.0, 110.0)
- added U2: SN65HVD72, Housings_SOIC:SOIC-8_3.9x4.9mm_Pitch1.27mm, F.Cu at (140.0, 134.5)
- added X1: 16MHz, Crystals:Crystal_HC49-SD_SMD, F.Cu at (120.0, 132.0)
Other:
- board outline added: 80 x 49 mm
