File: line-interface/line-interface.sch (KiCad schematic (older format))
At the start: 38 parts, among them IC1 ATTINY441-SSU, J1 CONN_01X06, P1 CONN_02X03, P2 CONN_01X04, Q1 NDT2955, U1 LR12K, U2 SN65HVD72, X1 16MHz

Commit message: Finish routing the board, manufacturing order sent
Connections:
- net labels removed: EXCITATION
- wire segments 68 -> 67
Changed lines of the file:
@@
 $EndComp
 $Comp
-L GND #PWR11
+L GND #PWR01
 U 1 1 58BAC83B
 P 5300 4700
-F 0 "#PWR11" H 5300 4450 60  0001 C CNN
+F 0 "#PWR01" H 5300 4450 60  0001 C CNN
 F 1 "GND" H 5300 4550 60  0000 C CNN
 F 2 "" H 5300 4700 60  0000 C CNN
@@
 $EndComp
 $Comp
-L VCC #PWR4
+L VCC #PWR02
 U 1 1 58BAC83C
 P 1200 1050
-F 0 "#PWR4" H 1200 900 60  0001 C CNN
+F 0 "#PWR02" H 1200 900 60  0001 C CNN
 F 1 "VCC" H 1200 1200 60  0000 C CNN
 F 2 "" H 1200 1050 60  0000 C CNN
@@
 $EndComp
 $Comp
-L GND #PWR3
+L GND #PWR03
 U 1 1 58BAC83D
 P 900 4500
-F 0 "#PWR3" H 900 4250 60  0001 C CNN
+F 0 "#PWR03" H 900 4250 60  0001 C CNN
 F 1 "GND" H 900 4350 60  0000 C CNN
 F 2 "" H 900 4500 60  0000 C CNN
@@
 $EndComp
 $Comp
-L GND #PWR2
+L GND #PWR04
 U 1 1 58BAC83F
 P 900 3600
-F 0 "#PWR2" H 900 3350 60  0001 C CNN
+F 0 "#PWR04" H 900 3350 60  0001 C CNN
 F 1 "GND" H 900 3450 60  0000 C CNN
 F 2 "" H 900 3600 60  0000 C CNN
@@
 $EndComp
 $Comp
-L GND #PWR20
+L GND #PWR05
 U 1 1 58BAC84B
 P 9800 3650
-F 0 "#PWR20" H 9800 3400 60  0001 C CNN
+F 0 "#PWR05" H 9800 3400 60  0001 C CNN
 F 1 "GND" H 9800 3500 60  0000 C CNN
 F 2 "" H 9800 3650 60  0000 C CNN
@@
 $EndComp
 $Comp
-L GND #PWR14
+L GND #PWR06
 U 1 1 58BAC84E
 P 6250 2850
-F 0 "#PWR14" H 6250 2600 60  0001 C CNN
+F 0 "#PWR06" H 6250 2600 60  0001 C CNN
 F 1 "GND" H 6250 2700 60  0000 C CNN
 F 2 "" H 6250 2850 60  0000 C CNN
@@
 $EndComp
 $Comp
-L GND #PWR12
+L GND #PWR07
 U 1 1 58BAC84F
 P 6000 4000
-F 0 "#PWR12" H 6000 3750 60  0001 C CNN
+F 0 "#PWR07" H 6000 3750 60  0001 C CNN
 F 1 "GND" H 6000 3850 60  0000 C CNN
 F 2 "" H 6000 4000 60  0000 C CNN
@@
 $EndComp
 $Comp
-L GND #PWR5
+L GND #PWR08
 U 1 1 58BAC852
 P 3850 4800
-F 0 "#PWR5" H 3850 4550 60  0001 C CNN
+F 0 "#PWR08" H 3850 4550 60  0001 C CNN
 F 1 "GND" H 3850 4650 60  0000 C CNN
 F 2 "" H 3850 4800 60  0000 C CNN
@@
 Text Label 3550 4500 2    60   ~ 0
 RESET
-Text Label 3550 4400 2    60   ~ 0
-EXCITATION
 Text Label 3300 3800 2    60   ~ 0
 MISO
@@
 	3000 4500 3850 4500
 Wire Wire Line
-	3000 4400 3550 4400
-Wire Wire Line
 	3000 3800 3300 3800
 Wire Wire Line
-	3500 4000 3000 4000
+	3300 4000 3000 4000
 Wire Wire Line
 	6400 3500 6900 3500
@@
 $EndComp
 $Comp
-L VCC #PWR17
+L VCC #PWR09
 U 1 1 58BAC858
 P 9550 4500
-F 0 "#PWR17" H 9550 4350 60  0001 C CNN
+F 0 "#PWR09" H 9550 4350 60  0001 C CNN
 F 1 "VCC" H 9550 4650 60  0000 C CNN
 F 2 "" H 9550 4500 60  0000 C CNN
@@
 $EndComp
 $Comp
-L GND #PWR18
+L GND #PWR010
 U 1 1 58BAC859
 P 9550 4800
-F 0 "#PWR18" H 9550 4550 60  0001 C CNN
+F 0 "#PWR010" H 9550 4550 60  0001 C CNN
 F 1 "GND" H 9550 4650 60  0000 C CNN
 F 2 "" H 9550 4800 60  0000 C CNN
@@
 $EndComp
 Wire Wire Line
+	9550 4700 8850 4700
+Text Label 8850 4700 0    60   ~ 0
+RS485A
+Wire Wire Line
 	9550 4600 8850 4600
 Text Label 8850 4600 0    60   ~ 0
-RS485A
-Wire Wire Line
-	9550 4700 8850 4700
-Text Label 8850 4700 0    60   ~ 0
 RS485B
 Connection ~ 3900 1350
@@
 $EndComp
 $Comp
-L GND #PWR8
+L GND #PWR011
 U 1 1 58BAC85B
 P 4300 2150
-F 0 "#PWR8" H 4300 1900 60  0001 C CNN
+F 0 "#PWR011" H 4300 1900 60  0001 C CNN
 F 1 "GND" H 4300 2000 60  0000 C CNN
 F 2 "" H 4300 2150 60  0000 C CNN
@@
 Connection ~ 9450 2600
 $Comp
-L GND #PWR16
+L GND #PWR012
 U 1 1 58BAE8F5
 P 9550 2700
-F 0 "#PWR16" H 9550 2450 60  0001 C CNN
+F 0 "#PWR012" H 9550 2450 60  0001 C CNN
 F 1 "GND" H 9550 2550 60  0000 C CNN
 F 2 "" H 9550 2700 60  0000 C CNN
@@
 Connection ~ 9550 2200
 $Comp
-L +5V #PWR15
+L +5V #PWR013
 U 1 1 58BAEA7B
 P 9450 1900
-F 0 "#PWR15" H 3500 550 50  0001 C CNN
+F 0 "#PWR013" H 3500 550 50  0001 C CNN
 F 1 "+5V" H 9465 2073 50  0000 C CNN
 F 2 "" H 3500 700 50  0001 C CNN
@@
 $EndComp
 $Comp
-L +5V #PWR13
+L +5V #PWR014
 U 1 1 58BAEAE2
 P 6250 2550
-F 0 "#PWR13" H 300 1200 50  0001 C CNN
+F 0 "#PWR014" H 300 1200 50  0001 C CNN
 F 1 "+5V" H 6265 2723 50  0000 C CNN
 F 2 "" H 300 1350 50  0001 C CNN
@@
 $EndComp
 $Comp
-L +5V #PWR1
+L +5V #PWR015
 U 1 1 58BAEBC4
 P 900 3300
-F 0 "#PWR1" H -5050 1950 50  0001 C CNN
+F 0 "#PWR015" H -5050 1950 50  0001 C CNN
 F 1 "+5V" H 915 3473 50  0000 C CNN
 F 2 "" H -5050 2100 50  0001 C CNN
@@
 $EndComp
 $Comp
-L +5V #PWR7
+L +5V #PWR016
 U 1 1 58BAED8C
 P 4150 4500
-F 0 "#PWR7" H -1800 3150 50  0001 C CNN
+F 0 "#PWR016" H -1800 3150 50  0001 C CNN
 F 1 "+5V" H 4250 4600 50  0000 C CNN
 F 2 "" H -1800 3300 50  0001 C CNN
@@
 Connection ~ 4300 1650
 $Comp
-L +5V #PWR10
+L +5V #PWR017
 U 1 1 58BB04F1
 P 5100 1200
-F 0 "#PWR10" H -850 -150 50  0001 C CNN
+F 0 "#PWR017" H -850 -150 50  0001 C CNN
 F 1 "+5V" H 5115 1373 50  0000 C CNN
 F 2 "" H -850 0   50  0001 C CNN
@@
 	0    1    1    0
 $EndComp
-Wire Wire Line
-	3500 3700 3500 4000
-$Comp
-L GND #PWR6
+$Comp
+L GND #PWR018
 U 1 1 58BD465C
 P 4050 4000
-F 0 "#PWR6" H 4050 3750 60  0001 C CNN
+F 0 "#PWR018" H 4050 3750 60  0001 C CNN
 F 1 "GND" H 4050 3850 60  0000 C CNN
 F 2 "" H 4050 4000 60  0000 C CNN
@@
 $EndComp
 Wire Wire Line
-	3000 3600 4150 3600
+	3000 3600 3500 3600
 Wire Wire Line
 	3800 3700 4450 3700
@@
 $EndComp
 $Comp
-L +5V #PWR19
+L +5V #PWR019
 U 1 1 58BD7C66
 P 9800 3450
-F 0 "#PWR19" H 3850 2100 50  0001 C CNN
+F 0 "#PWR019" H 3850 2100 50  0001 C CNN
 F 1 "+5V" H 9815 3623 50  0000 C CNN
 F 2 "" H 3850 2250 50  0001 C CNN
@@
 Connection ~ 4050 3700
 $Comp
-L +5V #PWR9
+L +5V #PWR020
 U 1 1 58BD9228
 P 4600 4000
-F 0 "#PWR9" H -1350 2650 50  0001 C CNN
+F 0 "#PWR020" H -1350 2650 50  0001 C CNN
 F 1 "+5V" H 4615 4173 50  0000 C CNN
 F 2 "" H -1350 2800 50  0001 C CNN
@@
 Wire Wire Line
 	4600 4000 4450 4000
-Text Label 4150 3600 2    60   ~ 0
+Text Label 3300 4000 2    60   ~ 0
 ~CS
+Wire Wire Line
+	3500 3600 3500 3700
 $EndSCHEMATC

Commit message: Add firmware of the line sensor, basic stuff -- it spits out sensor data in '1' and '0' ascii strings. Also hardware fixez: * P-channel mosfet has different numbering * a new regulator for power handling capabilities * correct pinout of rs485 transceiver * remove stupid led, what was I thinking?
Parts:
- removed D5: RED, LEDs:LED_0603, symbol LED_ALT
- removed R5: 18.2k, Resistors_SMD:R_0603_HandSoldering, symbol R
- removed R7: 6.04k, Resistors_SMD:R_0603_HandSoldering, symbol R
- removed U1: LR12K, TO_SOT_Packages_SMD:TO-252-2Lead, symbol LR12K-RESCUE-line-interface
- added U1: LM7805CT, TO_SOT_Packages_THT:TO-220_Horizontal, symbol LM7805CT
- Q1: symbol Q_PMOS_GSD -> Q_PMOS_GDS
Connections:
- wire segments 67 -> 68
Changed lines of the file:
@@
 Wire Wire Line
 	6400 3500 6900 3500
-Wire Wire Line
-	3000 3500 5600 3500
-Wire Wire Line
-	3000 3400 5600 3400
 Connection ~ 5600 3700
-Wire Wire Line
-	5600 3700 5600 3800
 Wire Wire Line
 	5600 3700 4900 3700
@@
 Connection ~ 6250 2550
 $Comp
-L Q_PMOS_GSD Q1
+L Q_PMOS_GDS Q1
 U 1 1 58BAC865
 P 2450 1450
@@
 	1    0    0    -1
 $EndComp
-$Comp
-L R R5
-U 1 1 58BB002C
-P 4300 1900
-F 0 "R5" V 4380 1900 50  0000 C CNN
-F 1 "18.2k" V 4307 1901 50  0000 C CNN
-F 2 "Resistors_SMD:R_0603_HandSoldering" V 4230 1900 30  0001 C CNN
-F 3 "" H 4300 1900 30  0000 C CNN
-F 4 "?" H 4300 1900 60  0001 C CNN "PartNo"
-F 5 "?" H 4300 1900 60  0001 C CNN "Manufacturer"
-F 6 "1469829" H 4300 1900 60  0001 C CNN "Distributor"
-	1    4300 1900
-	-1   0    0    1
-$EndComp
-Wire Wire Line
-	4300 2050 4300 2150
-Wire Wire Line
-	4300 1650 4300 1750
-$Comp
-L R R7
-U 1 1 58BB0271
-P 4550 1650
-F 0 "R7" V 4630 1650 50  0000 C CNN
-F 1 "6.04k" V 4557 1651 50  0000 C CNN
-F 2 "Resistors_SMD:R_0603_HandSoldering" V 4480 1650 30  0001 C CNN
-F 3 "" H 4550 1650 30  0000 C CNN
-F 4 "?" H 4550 1650 60  0001 C CNN "PartNo"
-F 5 "?" H 4550 1650 60  0001 C CNN "Manufacturer"
-F 6 "2059386" H 4550 1650 60  0001 C CNN "Distributor"
-	1    4550 1650
-	0    -1   1    0
-$EndComp
-Wire Wire Line
-	4300 1650 4400 1650
-Connection ~ 4300 1650
+Wire Wire Line
+	4300 1650 4300 2150
 $Comp
 L +5V #PWR017
@@
 $EndComp
 $Comp
-L LED_ALT D5
-U 1 1 58BD44C6
-P 4450 3850
-F 0 "D5" V 4488 3732 50  0000 R CNN
-F 1 "RED" V 4397 3732 50  0000 R CNN
-F 2 "LEDs:LED_0603" H 300 200 50  0001 C CNN
-F 3 "" H 300 200 50  0001 C CNN
-F 4 "?" H 4450 3850 60  0001 C CNN "PartNo"
-F 5 "?" H 4450 3850 60  0001 C CNN "Manufacturer"
-F 6 "?" H 4450 3850 60  0001 C CNN "Distributor"
-	1    4450 3850
-	0    1    1    0
-$EndComp
-$Comp
 L GND #PWR018
 U 1 1 58BD465C
@@
 Wire Wire Line
 	3000 3600 3500 3600
-Wire Wire Line
-	3800 3700 4450 3700
 Connection ~ 2900 1350
 Wire Wire Line
-	4700 950  4700 1650
-$Comp
-L LR12K-RESCUE-line-interface U1
-U 1 1 58BD94ED
-P 4300 1400
-F 0 "U1" H 4300 1717 50  0000 C CNN
-F 1 "LR12K" H 4300 1626 50  0000 C CNN
-F 2 "TO_SOT_Packages_SMD:TO-252-2Lead" H -100 100 50  0001 C CIN
-F 3 "" H -100 0   50  0001 C CNN
-F 4 "?" H 4300 1400 60  0001 C CNN "PartNo"
-F 5 "?" H 4300 1400 60  0001 C CNN "Manufacturer"
-F 6 "2448520" H 4300 1400 60  0001 C CNN "Distributor"
-	1    4300 1400
-	1    0    0    -1
-$EndComp
+	4700 950  4700 1350
 $Comp
 L Mounting_Hole MK1
@@
 Text Label 11150 2500 2    60   ~ 0
 ~CS
-Connection ~ 4050 3700
-$Comp
-L +5V #PWR020
-U 1 1 58BD9228
-P 4600 4000
-F 0 "#PWR020" H -1350 2650 50  0001 C CNN
-F 1 "+5V" H 4615 4173 50  0000 C CNN
-F 2 "" H -1350 2800 50  0001 C CNN
-F 3 "" H -1350 2800 50  0001 C CNN
-	1    4600 4000
-	1    0    0    -1
-$EndComp
-Wire Wire Line
-	4600 4000 4450 4000
 Text Label 3300 4000 2    60   ~ 0
 ~CS
 Wire Wire Line
 	3500 3600 3500 3700
+$Comp
+L LM7805CT U1
+U 1 1 58CBB2F0
+P 4300 1400
+F 0 "U1" H 4300 1717 50  0000 C CNN
+F 1 "LM7805CT" H 4300 1626 50  0000 C CNN
+F 2 "TO_SOT_Packages_THT:TO-220_Horizontal" H 4300 1500 50  0001 C CIN
+F 3 "" H 4300 1400 50  0001 C CNN
+F 4 "?" H 4300 1400 60  0001 C CNN "PartNo"
+F 5 "?" H 4300 1400 60  0001 C CNN "Manufacturer"
+F 6 "?" H 4300 1400 60  0001 C CNN "Distributor"
+	1    4300 1400
+	1    0    0    -1
+$EndComp
+Wire Wire Line
+	5600 3500 5600 3700
+Wire Wire Line
+	5600 3400 5000 3400
+Wire Wire Line
+	5000 3400 5000 3500
+Wire Wire Line
+	5000 3500 3000 3500
+Wire Wire Line
+	3000 3400 4800 3400
+Wire Wire Line
+	4800 3400 4800 3800
+Wire Wire Line
+	4800 3800 5600 3800
+Wire Wire Line
+	3800 3700 4050 3700
 $EndSCHEMATC

Commit message: Fix the line interface once more - input resistor has to be rated for 2W, also vias because no hole metallisation
Parts:
- R1: footprint Resistors_SMD:R_0805_HandSoldering -> Resistors_SMD:R_2512; Distributor 1738932 -> 9235892
Changed lines of the file:
@@
 F 0 "R1" V 1480 1350 50  0000 C CNN
 F 1 "10" V 1407 1351 50  0000 C CNN
-F 2 "Resistors_SMD:R_0805_HandSoldering" V 1330 1350 30  0001 C CNN
+F 2 "Resistors_SMD:R_2512" V 1330 1350 30  0001 C CNN
 F 3 "" H 1400 1350 30  0000 C CNN
 F 4 "?" H 1400 1350 60  0001 C CNN "PartNo"
 F 5 "?" H 1400 1350 60  0001 C CNN "Manufacturer"
-F 6 "1738932" H 1400 1350 60  0001 C CNN "Distributor"
+F 6 "9235892" H 1400 1350 60  0001 C CNN "Distributor"
 	1    1400 1350
 	0    -1   -1   0
