File: controller/steering-wheel-takeover.sch (KiCad schematic (older format))
At the start: 29 parts, among them J10 CONN_01X02, J11 CONN_01X02, J12 CONN_01X02, J7 CONN_01X02, J8 CONN_01X02, J9 CONN_01X02, K10 RELAY_SEPARATED, K11 RELAY_SEPARATED, K12 RELAY_SEPARATED, K7 RELAY_SEPARATED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

Commit message: Start putting the controller together, add various subsystems
Other:
- note added: "TODO: SĖDYNĖ"
Changed lines of the file:
@@
 Text HLabel 1850 2050 0    60   Input ~ 0
 TAKEOVER_PEDAL
-Text Notes 10850 4550 0    60   ~ 0
+Text Notes 11900 4650 0    60   ~ 0
 TODO: ŠVIESOS
-Text Notes 10850 5150 0    60   ~ 0
+Text Notes 11900 5100 0    60   ~ 0
 TODO: MIRGALKĖ
-Text Notes 10300 1450 0    60   ~ 0
+Text Notes 11800 1400 0    60   ~ 0
 TODO: RAKTELIS
 $Comp
@@
 Text HLabel 9550 850  0    60   Input ~ 0
 STEERING_COMMON
+Text Notes 11900 4100 0    60   ~ 0
+TODO: SĖDYNĖ
 $EndSCHEMATC
