File: controller/controller.kicad_pcb (KiCad board)
At the start: 2 copper layers, 0 parts

Commit message: Some progress with controller board routing
Parts:
- added C1: C, Capacitors_SMD:C_0603_HandSoldering, B.Cu at (46.0, 38.5)
- added C10: C, Capacitors_SMD:C_0603_HandSoldering, B.Cu at (215.1, 38.5)
- added C11: C, Capacitors_SMD:C_0603_HandSoldering, B.Cu at (225.0, 38.5)
- added C12: C, Capacitors_SMD:C_0603_HandSoldering, B.Cu at (234.9, 38.5)
- added C13: C, Capacitors_SMD:C_0603_HandSoldering, B.Cu at (149.4, 38.5)
- added C14: C, Capacitors_SMD:C_0603_HandSoldering, B.Cu at (159.6, 38.5)
- added C15: 470u, Capacitors_ThroughHole:CP_Radial_D16.0mm_P7.50mm, F.Cu at (37.2, 36.5)
- added C16: C, Capacitors_SMD:C_1210_HandSoldering, F.Cu at (136.5, 38.0)
- added C17: C, Capacitors_SMD:C_0603_HandSoldering, B.Cu at (120.0, 38.5)
- added C18: C, Capacitors_SMD:C_0603_HandSoldering, B.Cu at (169.6, 38.5)
- added C19: C, Capacitors_SMD:C_0603_HandSoldering, B.Cu at (179.4, 38.5)
- added C2: C, Capacitors_SMD:C_0603_HandSoldering, B.Cu at (56.0, 38.5)
- added C20: 1u, Capacitors_SMD:C_0603_HandSoldering, F.Cu at (66.8, 205.9)
- added C21: C, Capacitors_SMD:C_0603_HandSoldering, F.Cu at (201.9, 153.4)
- added C22: C, Capacitors_SMD:C_0603_HandSoldering, B.Cu at (204.5, 53.0)
- added C23: C, Capacitors_SMD:C_0603_HandSoldering, B.Cu at (46.0, 56.0)
- added C24: C, Capacitors_SMD:C_0603_HandSoldering, B.Cu at (56.0, 56.0)
- added C25: C, Capacitors_SMD:C_0603_HandSoldering, B.Cu at (66.0, 56.0)
- added C26: C, Capacitors_SMD:C_0603_HandSoldering, B.Cu at (76.0, 56.0)
- added C27: C, Capacitors_SMD:C_0603_HandSoldering, B.Cu at (86.0, 56.0)
- added C28: C, Capacitors_SMD:C_0603_HandSoldering, B.Cu at (159.6, 56.0)
- added C29: C, Capacitors_SMD:C_0603_HandSoldering, B.Cu at (120.0, 56.0)
- added C3: C, Capacitors_SMD:C_0603_HandSoldering, B.Cu at (66.0, 38.5)
- added C30: C, Capacitors_SMD:C_0603_HandSoldering, B.Cu at (130.1, 56.0)
- added C31: C, Capacitors_SMD:C_0603_HandSoldering, B.Cu at (149.4, 56.0)
- added C32: C, Capacitors_SMD:C_0603_HandSoldering, B.Cu at (129.9, 38.5)
- added C33: C, Capacitors_SMD:C_0603_HandSoldering, F.Cu at (178.4, 163.1)
- added C34: 470u, Capacitors_ThroughHole:CP_Radial_D16.0mm_P7.50mm, F.Cu at (33.0, 208.7)
- added C35: 1u, Capacitors_SMD:C_0603_HandSoldering, F.Cu at (51.7, 217.9)
- added C36: 1u, Capacitors_SMD:C_1210_HandSoldering, F.Cu at (193.3, 189.6)
- added C37: 470u, Capacitors_ThroughHole:CP_Radial_D16.0mm_P7.50mm, F.Cu at (194.6, 168.3)
- added C38: 1u, Capacitors_SMD:C_1210_HandSoldering, F.Cu at (200.2, 189.6)
- added C39: 1u, Capacitors_SMD:C_0603, F.Cu at (245.7, 171.1)
- added C4: C, Capacitors_SMD:C_0603_HandSoldering, B.Cu at (76.0, 38.5)
- added C40: 470u, Capacitors_ThroughHole:CP_Radial_D16.0mm_P7.50mm, F.Cu at (150.9, 160.8)
- added C41: 470u, Capacitors_ThroughHole:CP_Radial_D16.0mm_P7.50mm, F.Cu at (133.7, 160.8)
- added C42: 470u, Capacitors_ThroughHole:CP_Radial_D16.0mm_P7.50mm, F.Cu at (115.7, 183.0)
- added C43: 470u, Capacitors_ThroughHole:CP_Radial_D16.0mm_P7.50mm, F.Cu at (33.0, 160.8)
- added C44: C, Capacitors_SMD:C_1210_HandSoldering, F.Cu at (31.7, 189.9)
- added C5: C, Capacitors_SMD:C_0603_HandSoldering, B.Cu at (86.0, 38.5)
- added C6: C, Capacitors_SMD:C_0603_HandSoldering, B.Cu at (95.5, 38.5)
- added C7: 470u, Capacitors_ThroughHole:CP_Radial_D16.0mm_P7.50mm, F.Cu at (264.0, 31.0)
- added C8: C, Capacitors_SMD:C_1210_HandSoldering, F.Cu at (270.0, 33.0)
- added C9: C, Capacitors_SMD:C_0603_HandSoldering, B.Cu at (205.1, 38.5)
- added D1: D_ALT, Diodes_SMD:D_SOD-123, B.Cu at (45.9, 36.5)
- added D10: D_ALT, Diodes_SMD:D_SOD-123, B.Cu at (235.0, 36.5)
- added D11: D_ALT, Diodes_SMD:D_SOD-123, B.Cu at (149.3, 36.5)
- added D12: D_ALT, Diodes_SMD:D_SOD-123, B.Cu at (159.3, 36.5)
- added D13: D_ALT, Diodes_SMD:D_SOD-123, B.Cu at (119.8, 36.5)
- added D14: D_ALT, Diodes_SMD:D_SOD-123, B.Cu at (169.3, 36.5)
- added D15: D_ALT, Diodes_SMD:D_SOD-123, B.Cu at (179.3, 36.5)
- added D16: 5V, Diodes_SMD:SOD-123, F.Cu at (197.4, 149.1)
- added D17: D_ALT, Diodes_SMD:D_SOD-123, B.Cu at (206.2, 51.0)
- added D18: D_ALT, Diodes_SMD:D_SOD-123, B.Cu at (45.6, 54.0)
- added D19: D_ALT, Diodes_SMD:D_SOD-123, B.Cu at (55.9, 54.0)
- added D2: D_ALT, Diodes_SMD:D_SOD-123, B.Cu at (55.9, 36.5)
- added D20: D_ALT, Diodes_SMD:D_SOD-123, B.Cu at (66.2, 54.0)
- added D21: D_ALT, Diodes_SMD:D_SOD-123, B.Cu at (76.2, 54.0)
- added D22: D_ALT, Diodes_SMD:D_SOD-123, B.Cu at (85.8, 54.5)
- added D23: D_ALT, Diodes_SMD:D_SOD-123, B.Cu at (159.7, 54.5)
- added D24: D_ALT, Diodes_SMD:D_SOD-123, B.Cu at (120.0, 54.5)
- added D25: D_ALT, Diodes_SMD:D_SOD-123, B.Cu at (129.9, 54.5)
- added D26: D_ALT, Diodes_SMD:D_SOD-123, B.Cu at (149.3, 54.5)
- added D27: D_ALT, Diodes_SMD:D_SOD-123, B.Cu at (130.1, 36.5)
- added D28: 16V, Diodes_SMD:D_SMB_Handsoldering, F.Cu at (268.8, 37.5)
- added D29: 16V, Diodes_SMD:D_SMB_Handsoldering, B.Cu at (39.5, 33.5)
- added D3: D_ALT, Diodes_SMD:D_SOD-123, B.Cu at (65.8, 36.5)
- added D30: LED_Small_ALT, LEDs:LED_0805, F.Cu at (168.9, 153.2)
- added D31: LED_Small_ALT, LEDs:LED_0805, F.Cu at (133.8, 189.9)
- added D32: LED_Small_ALT, LEDs:LED_0805, F.Cu at (148.2, 173.4)
- added D33: LED_Small_ALT, LEDs:LED_0805, F.Cu at (148.2, 178.5)
- added D34: D_TVS_ALT, Diodes_SMD:Diode-SMC_Handsoldering, F.Cu at (213.8, 164.3)
- added D35: LED_Small_ALT, LEDs:LED_D5.0mm, F.Cu at (93.3, 130.5)
- added D36: LED_Small_ALT, LEDs:LED_D5.0mm, F.Cu at (69.5, 134.1)
- added D37: LED_Small_ALT, LEDs:LED_D5.0mm, F.Cu at (101.2, 120.4)
- added D38: LED_Small_ALT, LEDs:LED_D5.0mm, F.Cu at (106.1, 109.6)
- added D39: LED_Small_ALT, LEDs:LED_D5.0mm, F.Cu at (117.5, 104.6)
- added D4: D_ALT, Diodes_SMD:D_SOD-123, B.Cu at (76.0, 36.5)
- added D40: LED_Small_ALT, LEDs:LED_D5.0mm, F.Cu at (106.1, 114.7)
- added D41: LED_Small_ALT, LEDs:LED_D5.0mm, F.Cu at (89.7, 125.4)
- added D42: LED_Small_ALT, LEDs:LED_D5.0mm, F.Cu at (159.4, 65.5)
- added D43: LED_Small_ALT, LEDs:LED_D5.0mm, F.Cu at (44.7, 63.1)
- added D44: LED_Small_ALT, LEDs:LED_D5.0mm, F.Cu at (55.1, 63.1)
- added D45: LED_Small_ALT, LEDs:LED_D5.0mm, F.Cu at (64.7, 63.1)
- added D46: LED_Small_ALT, LEDs:LED_D5.0mm, F.Cu at (74.7, 63.1)
- added D47: LED_Small_ALT, LEDs:LED_D5.0mm, F.Cu at (84.6, 63.1)
- added D48: LED_Small_ALT, LEDs:LED_D5.0mm, F.Cu at (151.0, 63.0)
- added D49: LED_Small_ALT, LEDs:LED_D5.0mm, F.Cu at (131.2, 63.1)
- added D5: D_ALT, Diodes_SMD:D_SOD-123, B.Cu at (85.7, 36.5)
- added D50: LED_Small_ALT, LEDs:LED_D5.0mm, F.Cu at (121.2, 63.1)
- added D51: LED_Small_ALT, LEDs:LED_0805, F.Cu at (133.8, 184.8)
- added D52: 16V, Diodes_SMD:D_SMB_Handsoldering, F.Cu at (239.1, 173.7)
- added D53: 16V, Diodes_SMD:D_SMB_Handsoldering, F.Cu at (236.8, 184.1)
- added D54: D, Diodes_SMD:D_SOD-123, F.Cu at (206.3, 189.3)
- added D55: GREEN, LEDs:LED_0603, F.Cu at (248.3, 165.9)
- added D56: 16V, Diodes_SMD:D_SMB_Handsoldering, F.Cu at (147.4, 185.2)
- added D57: 16V, Diodes_SMD:D_SMB_Handsoldering, F.Cu at (158.9, 175.1)
- added D58: 16V, Diodes_SMD:D_SMB_Handsoldering, F.Cu at (47.1, 186.2)
- added D6: D_ALT, Diodes_SMD:D_SOD-123, B.Cu at (95.5, 36.5)
- added D7: D_ALT, Diodes_SMD:D_SOD-123, B.Cu at (204.8, 36.5)
- added D8: D_ALT, Diodes_SMD:D_SOD-123, B.Cu at (214.8, 36.5)
- added D9: D_ALT, Diodes_SMD:D_SOD-123, B.Cu at (224.8, 36.5)
- added F1: Fuse, smalsiukas-footpints:Automotive-Fuse-Holder, F.Cu at (55.1, 202.5)
- added F2: Fuse, smalsiukas-footpints:Automotive-Fuse-Holder, F.Cu at (199.5, 182.2)
- added J1: CONN_01X10, Connectors_Terminal_Blocks:TerminalBlock_Pheonix_MKDS1.5-10pol, F.Cu at (33.5, 23.0)
- added J2: CONN_01X10, Connectors_Terminal_Blocks:TerminalBlock_Pheonix_MKDS1.5-10pol, F.Cu at (86.0, 23.0)
- added J3: CONN_01X10, Connectors_Terminal_Blocks:TerminalBlock_Pheonix_MKDS1.5-10pol, F.Cu at (138.5, 23.0)
- added J4: CONN_01X10, Connectors_Terminal_Blocks:TerminalBlock_Pheonix_MKDS1.5-10pol, F.Cu at (191.0, 23.0)
- added K1: RELAY_SEPARATED, smalsiukas-footpints:Relay_SPDT, F.Cu at (48.5, 41.0)
- added K10: RELAY_SEPARATED, smalsiukas-footpints:Relay_SPDT, F.Cu at (217.5, 41.0)
- added K11: RELAY_SEPARATED, smalsiukas-footpints:Relay_SPDT, F.Cu at (227.5, 41.0)
- added K12: RELAY_SEPARATED, smalsiukas-footpints:Relay_SPDT, F.Cu at (237.5, 41.0)
- added K13: RELAY_SEPARATED, smalsiukas-footpints:Relay_SPDT, F.Cu at (152.0, 41.0)
- added K14: RELAY_SEPARATED, smalsiukas-footpints:Relay_SPDT, F.Cu at (162.0, 41.0)
- added K15: RELAY_SEPARATED, smalsiukas-footpints:Relay_SPDT, F.Cu at (172.0, 41.0)
- added K16: RELAY_SEPARATED, smalsiukas-footpints:Relay_SPDT, F.Cu at (182.0, 41.0)
- added K17: RELAY_SEPARATED, smalsiukas-footpints:Relay_SPDT, F.Cu at (207.5, 58.5)
- added K18: RELAY_SEPARATED, smalsiukas-footpints:Relay_SPDT, F.Cu at (48.5, 58.5)
- added K19: RELAY_SEPARATED, smalsiukas-footpints:Relay_SPDT, F.Cu at (58.5, 58.5)
- added K2: RELAY_SEPARATED, smalsiukas-footpints:Relay_SPDT, F.Cu at (58.5, 41.0)
- added K20: RELAY_SEPARATED, smalsiukas-footpints:Relay_SPDT, F.Cu at (68.5, 58.5)
- added K21: RELAY_SEPARATED, smalsiukas-footpints:Relay_SPDT, F.Cu at (78.5, 58.5)
- added K22: RELAY_SEPARATED, smalsiukas-footpints:Relay_SPDT, F.Cu at (88.5, 58.5)
- added K23: RELAY_SEPARATED, smalsiukas-footpints:Relay_SPDT, F.Cu at (162.0, 58.5)
- added K24: RELAY_SEPARATED, smalsiukas-footpints:Relay_SPDT, F.Cu at (122.5, 58.5)
- added K25: RELAY_SEPARATED, smalsiukas-footpints:Relay_SPDT, F.Cu at (132.5, 58.5)
- added K26: RELAY_SEPARATED, smalsiukas-footpints:Relay_SPDT, F.Cu at (152.0, 58.5)
- added K3: RELAY_SEPARATED, smalsiukas-footpints:Relay_SPDT, F.Cu at (68.5, 41.0)
- added K4: RELAY_SEPARATED, smalsiukas-footpints:Relay_SPDT, F.Cu at (78.5, 41.0)
- added K5: RELAY_SEPARATED, smalsiukas-footpints:Relay_SPDT, F.Cu at (88.5, 41.0)
- added K6: RELAY_SEPARATED, smalsiukas-footpints:Relay_SPDT, F.Cu at (98.1, 41.0)
- added K7: RELAY_SEPARATED, smalsiukas-footpints:Relay_SPDT, F.Cu at (122.5, 41.0)
- added K8: RELAY_SEPARATED, smalsiukas-footpints:Relay_SPDT, F.Cu at (132.5, 41.0)
- added K9: RELAY_SEPARATED, smalsiukas-footpints:Relay_SPDT, F.Cu at (207.5, 41.0)
- added MK1: Mounting_Hole, Mounting_Holes:MountingHole_3.2mm_M3, F.Cu at (283.1, 122.1)
- added MK2: Mounting_Hole, Mounting_Holes:MountingHole_3.2mm_M3, F.Cu at (327.1, 114.0)
- added MK3: Mounting_Hole, Mounting_Holes:MountingHole_3.2mm_M3, F.Cu at (327.1, 103.6)
- added MK4: Mounting_Hole, Mounting_Holes:MountingHole_3.2mm_M3, F.Cu at (294.5, 122.1)
- added MK5: Mounting_Hole, Mounting_Holes:MountingHole_3.2mm_M3, F.Cu at (214.9, 187.0)
- added MK6: Mounting_Hole, Mounting_Holes:MountingHole_3.2mm_M3, F.Cu at (239.9, 163.4)
- added MK7: Mounting_Hole, Mounting_Holes:MountingHole_3.2mm_M3, F.Cu at (226.2, 187.0)
- added MK8: Mounting_Hole, Mounting_Holes:MountingHole_3.2mm_M3, F.Cu at (228.5, 174.8)
- added Q1: Q_NMOS_GSD, Housings_SOT-23_SOT-143_TSOT-6:SOT-23_Handsoldering, F.Cu at (200.0, 136.0)
- added Q2: Q_NMOS_GSD, TO_SOT_Packages_SMD:SOT-23_Handsoldering, F.Cu at (243.2, 116.0)
- added Q3: Q_PMOS_GSD, TO_SOT_Packages_SMD:SOT-23_Handsoldering, F.Cu at (235.3, 130.1)
- added Q4: Q_NMOS_GSD, TO_SOT_Packages_SMD:SOT-23_Handsoldering, F.Cu at (225.1, 131.6)
- added Q5: Q_PMOS_GSD, TO_SOT_Packages_SMD:SOT-23_Handsoldering, F.Cu at (243.2, 123.0)
- added Q6: Q_PMOS_GSD, TO_SOT_Packages_SMD:SOT-23_Handsoldering, F.Cu at (253.5, 116.0)
- added Q7: Q_NMOS_GSD, TO_SOT_Packages_SMD:TO-252-2Lead, F.Cu at (134.8, 176.5)
- added Q8: NDT2955, TO_SOT_Packages_SMD:TO-252-2Lead, F.Cu at (215.1, 175.9)
- added Q9: Q_NMOS_GSD, Housings_SOT-23_SOT-143_TSOT-6:SOT-23_Handsoldering, F.Cu at (77.5, 203.4)
- added R1: 100k, Resistors_SMD:R_0603_HandSoldering, F.Cu at (265.4, 110.9)
- added R10: 100k, Resistors_SMD:R_0603_HandSoldering, F.Cu at (250.5, 122.0)
- added R11: 0, Resistors_SMD:R_0603_HandSoldering, F.Cu at (240.4, 136.1)
- added R12: R, Resistors_SMD:R_0603_HandSoldering, F.Cu at (165.4, 166.1)
- added R13: R, Resistors_SMD:R_0603_HandSoldering, F.Cu at (156.2, 183.3)
- added R14: R, Resistors_SMD:R_0603_HandSoldering, F.Cu at (176.9, 153.2)
- added R15: R, Resistors_SMD:R_0603_HandSoldering, F.Cu at (175.9, 158.3)
- added R16: R, Resistors_SMD:R_0603_HandSoldering, F.Cu at (174.2, 163.3)
- added R17: R, Resistors_SMD:R_0603_HandSoldering, F.Cu at (171.5, 158.3)
- added R18: 1k, Resistors_SMD:R_0603_HandSoldering, F.Cu at (166.0, 171.2)
- added R19: R, Resistors_SMD:R_0603_HandSoldering, F.Cu at (154.6, 188.4)
- added R2: 100k, Resistors_SMD:R_0603_HandSoldering, F.Cu at (259.2, 125.0)
- added R21: R, Resistors_SMD:R_0603_HandSoldering, F.Cu at (170.4, 171.2)
- added R22: R, Resistors_SMD:R_0603_HandSoldering, F.Cu at (166.0, 176.2)
- added R23: R, Resistors_SMD:R_0603_HandSoldering, F.Cu at (117.0, 134.9)
- added R24: R, Resistors_SMD:R_0603_HandSoldering, F.Cu at (121.4, 129.8)
- added R25: R, Resistors_SMD:R_0603_HandSoldering, F.Cu at (126.5, 124.8)
- added R26: R, Resistors_SMD:R_0603_HandSoldering, F.Cu at (117.0, 129.8)
- added R27: R, Resistors_SMD:R_0603_HandSoldering, F.Cu at (125.7, 129.8)
- added R28: R, Resistors_SMD:R_0603_HandSoldering, F.Cu at (112.7, 134.9)
- added R29: R, Resistors_SMD:R_0603_HandSoldering, F.Cu at (125.4, 104.6)
- added R3: 1k, Resistors_SMD:R_0603_HandSoldering, F.Cu at (242.6, 129.0)
- added R30: R, Resistors_SMD:R_0603_HandSoldering, F.Cu at (117.8, 124.8)
- added R31: R, Resistors_SMD:R_0603_HandSoldering, F.Cu at (105.6, 135.5)
- added R32: R, Resistors_SMD:R_0603_HandSoldering, F.Cu at (112.7, 129.8)
- added R33: R, Resistors_SMD:R_0603_HandSoldering, F.Cu at (159.4, 62.9)
- added R34: R, Resistors_SMD:R_0603_HandSoldering, B.Cu at (46.6, 58.7)
- added R35: R, Resistors_SMD:R_0603_HandSoldering, B.Cu at (56.9, 58.7)
- added R36: R, Resistors_SMD:R_0603_HandSoldering, B.Cu at (66.6, 58.6)
- added R37: R, Resistors_SMD:R_0603_HandSoldering, B.Cu at (76.8, 58.6)
- added R38: R, Resistors_SMD:R_0603_HandSoldering, B.Cu at (86.7, 58.6)
- added R39: R, Resistors_SMD:R_0603_HandSoldering, B.Cu at (148.5, 58.6)
- added R4: 3.6k, Resistors_SMD:R_0603_HandSoldering, F.Cu at (260.7, 114.9)
- added R40: R, Resistors_SMD:R_0603_HandSoldering, B.Cu at (129.1, 58.4)
- added R41: R, Resistors_SMD:R_0603_HandSoldering, B.Cu at (119.2, 58.5)
- added R42: 330, Resistors_SMD:R_0603_HandSoldering, F.Cu at (254.8, 122.0)
- added R43: 100k, Resistors_SMD:R_0603_HandSoldering, F.Cu at (236.0, 136.1)
- added R44: 100k, Resistors_SMD:R_0603_HandSoldering, F.Cu at (269.5, 116.0)
- added R45: 100k, Resistors_SMD:R_0603_HandSoldering, F.Cu at (269.7, 100.8)
- added R46: 100k, Resistors_SMD:R_0603_HandSoldering, F.Cu at (265.1, 116.0)
- added R47: 330, Resistors_SMD:R_0603_HandSoldering, F.Cu at (254.8, 127.0)
- added R48: 330, Resistors_SMD:R_0603_HandSoldering, F.Cu at (247.0, 132.1)
- added R49: 100k, Resistors_SMD:R_0603_HandSoldering, F.Cu at (269.7, 110.9)
- added R5: R, Resistors_SMD:R_0603_HandSoldering, F.Cu at (206.4, 148.6)
- added R50: 100k, Resistors_SMD:R_0603_HandSoldering, F.Cu at (260.7, 120.0)
- added R51: 100k, Resistors_SMD:R_0603_HandSoldering, F.Cu at (265.4, 100.8)
- added R52: 100k, Resistors_SMD:R_0603_HandSoldering, F.Cu at (265.4, 105.9)
- added R53: 100k, Resistors_SMD:R_0603_HandSoldering, F.Cu at (227.3, 137.6)
- added R54: 169R, Resistors_SMD:R_0603_HandSoldering, F.Cu at (169.8, 166.1)
- added R55: R, Resistors_SMD:R_0603_HandSoldering, F.Cu at (180.2, 158.3)
- added R56: 100k, Resistors_SMD:R_0603_HandSoldering, F.Cu at (181.2, 153.2)
- added R57: 1k, Resistors_SMD:R_0603_HandSoldering, F.Cu at (66.9, 201.1)
- added R58: 1k, Resistors_SMD:R_0603_HandSoldering, F.Cu at (56.8, 209.0)
- added R59: 100k, Resistors_SMD:R_0603_HandSoldering, F.Cu at (47.5, 218.1)
- added R6: R, Resistors_SMD:R_0603_HandSoldering, F.Cu at (202.0, 148.6)
- added R60: 10k, Resistors_SMD:R_0603, F.Cu at (249.2, 175.8)
- added R61: 10, Resistors_SMD:R_0805_HandSoldering, F.Cu at (248.1, 160.9)
- added R62: 330, Resistors_SMD:R_0603, F.Cu at (249.2, 170.8)
- added R63: 169R, Resistors_SMD:R_0603_HandSoldering, F.Cu at (93.6, 206.1)
- added R64: 100k, Resistors_SMD:R_0603_HandSoldering, F.Cu at (89.2, 201.1)
- added R65: 330, Resistors_SMD:R_0603_HandSoldering, F.Cu at (89.2, 206.1)
- added R66: 330, Resistors_SMD:R_0603_HandSoldering, F.Cu at (93.6, 201.1)
- added R67: 330, Resistors_SMD:R_0603_HandSoldering, F.Cu at (84.8, 206.1)
- added R68: 1k, Resistors_SMD:R_0603_HandSoldering, F.Cu at (84.8, 201.1)
- added R7: 330, Resistors_SMD:R_0603_HandSoldering, F.Cu at (269.7, 105.9)
- added R8: 330, Resistors_SMD:R_0603_HandSoldering, F.Cu at (231.7, 137.6)
- added R9: 330, Resistors_SMD:R_0603_HandSoldering, F.Cu at (250.5, 127.0)
- added R91: R, Resistors_SMD:R_0603_HandSoldering, B.Cu at (111.4, 47.5)
- added R92: R, Resistors_SMD:R_0603_HandSoldering, B.Cu at (197.1, 47.5)
- added RN1: R_Network08, Resistors_THT:R_Array_SIP9, F.Cu at (178.2, 87.5)
- added RN2: R_Pack08, Resistors_SMD:R_Array_Convex_8x0602, B.Cu at (113.9, 55.4)
- added RV1: 40k, Potentiometers:Potentiometer_Trimmer_Bourns_3296P, F.Cu at (201.9, 121.6)
- added RV2: 40k, Potentiometers:Potentiometer_Trimmer_Bourns_3296P, F.Cu at (218.6, 118.5)
- added RV3: 40k, Potentiometers:Potentiometer_Trimmer_Bourns_3296P, F.Cu at (245.1, 102.9)
- added RV4: 40k, Potentiometers:Potentiometer_Trimmer_Bourns_3296P, F.Cu at (214.5, 132.6)
- added RV5: 40k, Potentiometers:Potentiometer_Trimmer_Bourns_3296P, F.Cu at (257.7, 102.9)
- added RV6: 40k, Potentiometers:Potentiometer_Trimmer_Bourns_3296P, F.Cu at (232.6, 102.9)
- added RV7: 40k, Potentiometers:Potentiometer_Trimmer_Bourns_3296P, F.Cu at (232.6, 116.9)
- added SH1: ARDUINO_NANO, w_conn_misc:arduino_nano_header, F.Cu at (299.4, 107.7)
- added U1: OPTO-TRANSISTOR-4, Housings_DIP:DIP-4_W11.48mm_SMD, F.Cu at (215.2, 103.8)
- added U10: ULN2803A, Housings_SOIC:SOIC-18W_7.5x11.6mm_Pitch1.27mm, B.Cu at (191.3, 78.1)
- added U11: ULN2803A, Housings_SOIC:SOIC-18W_7.5x11.6mm_Pitch1.27mm, B.Cu at (104.3, 56.2)
- added U12: OPTO-TRANSISTOR-4, Housings_DIP:DIP-4_W11.48mm_SMD, F.Cu at (203.2, 112.4)
- added U2: ULN2801A, Housings_SOIC:SOIC-18W_7.5x11.6mm_Pitch1.27mm, B.Cu at (193.7, 40.6)
- added U3: SN65HVD72, Housings_SOIC:SOIC-8_3.9x4.9mm_Pitch1.27mm, F.Cu at (50.0, 211.1)
- added U5: LM7805CT, TO_SOT_Packages_SMD:TO-252-2Lead, F.Cu at (226.5, 163.7)
- added U6: ULN2801A, Housings_SOIC:SOIC-18W_7.5x11.6mm_Pitch1.27mm, B.Cu at (109.8, 40.6)
- added U7: 74LS04, TO_SOT_Packages_SMD:SOT-23-5_HandSoldering, F.Cu at (166.3, 159.7)
- added U8: VNH3SP30, smalsiukas-footpints:SOIC-30, F.Cu at (120.7, 161.9)
- added U9: 74HC595, Housings_SOIC:SOIC-16_3.9x9.9mm_Pitch1.27mm, B.Cu at (104.2, 68.7)
Routing:
- net VCC: track 0.00 -> 319.6 mm, vias 0 -> 1
- net /Control Switching/~AUX_ENABLE_PWR: track 0.00 -> 82.5 mm
- net /Control Switching/~DIR_FWD_ENABLE_PWR: track 0.00 -> 77.7 mm
- net Net-(C1-Pad2): track 0.00 -> 70.0 mm
- net /ControlHacks/STEERING_COMMON: track 0.00 -> 69.6 mm
- net Net-(C2-Pad2): track 0.00 -> 59.8 mm
- net /Control Switching/~DIR_BACK_ENABLE_PWR: track 0.00 -> 59.8 mm
- net /Control Switching/~MIRGALKE_ENABLE_PWR: track 0.00 -> 59.2 mm
- net /Control Switching/~HORN_ENABLE_PWR: track 0.00 -> 57.2 mm
- net Net-(C13-Pad2): track 0.00 -> 53.7 mm
- net Net-(C3-Pad2): track 0.00 -> 49.7 mm
- net /ControlHacks/LIGHTS_COMMON: track 0.00 -> 47.3 mm
- net /Control Switching/~PARKING_DISABLE_PWR: track 0.00 -> 46.3 mm
- net /Control Switching/~LIGHTS_ENABLE_PWR: track 0.00 -> 46.0 mm
- net Net-(C14-Pad2): track 0.00 -> 43.4 mm
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