File: controller/Linde_steering/Linde_steering.kicad_pcb (KiCad board)
At the start: 2 copper layers, 21 parts, among them P1 CONN_01X06, P2 CONN_01X06, Q1 Q_NMOS_GDS, U1 LTV-827, U2 TL072

Commit message: Cleanup
Parts:
- D1, D2: value 6V8 -> BZX84V006.8; footprint Diodes_SMD:D_SMA_Handsoldering -> TO_SOT_Packages_SMD:SOT-23
- moved D2 5.09 mm to (152.7, 159.3), turned to 90 degrees
- moved D1 0.46 mm to (157.7, 159.3), turned to 90 degrees
Connections:
- D1 pad 1: Net-(D1-Pad1) -> GND
- D1 pad 2: GND -> (no net)
- D2 pad 1: Net-(D2-Pad1) -> GND
- D2 pad 2: GND -> (no net)
- P2 pad 3: Net-(D2-Pad1) -> Net-(D2-Pad3)
- P2 pad 4: Net-(D1-Pad1) -> Net-(D1-Pad3)
- U2 pad 1: Net-(D2-Pad1) -> Net-(D2-Pad3)
- U2 pad 2: Net-(D2-Pad1) -> Net-(D2-Pad3)
- U2 pad 6: Net-(D1-Pad1) -> Net-(D1-Pad3)
- U2 pad 7: Net-(D1-Pad1) -> Net-(D1-Pad3)
Routing:
- net Net-(D1-Pad1): track 22.0 -> 0.00 mm
- net Net-(D2-Pad1): track 20.7 -> 0.00 mm
- net Net-(D1-Pad3): track 0.00 -> 19.6 mm
- net Net-(D2-Pad3): track 0.00 -> 17.8 mm
- net GND: track 89.4 -> 95.4 mm
- net +5V: track 50.0 -> 50.9 mm

Commit message: Mounting holes added
Parts:
- added MK1: Mounting_Hole, Mounting_Holes:MountingHole_3.2mm_M3_Pad, F.Cu at (130.0, 135.0)
- added MK2: Mounting_Hole, Mounting_Holes:MountingHole_3.2mm_M3_Pad, F.Cu at (180.0, 135.0)
- added MK3: Mounting_Hole, Mounting_Holes:MountingHole_3.2mm_M3_Pad, F.Cu at (130.0, 160.0)
- added MK4: Mounting_Hole, Mounting_Holes:MountingHole_3.2mm_M3_Pad, F.Cu at (180.0, 160.0)
- moved R5 3.19 mm to (168.0, 159.3), turned to 180 degrees
Routing:
- net GND: track 95.4 -> 127.7 mm
- net Net-(R5-Pad1): track 24.7 -> 28.5 mm

Commit message: Cleanup
SMT GDS FET changed to more common GSD FET;
OSHW and CC symbols added to copper layer;
Gerbers updated and sent for manufacturing;

Typeo fixed in Arduino code
Parts:
- added REF**: Symbol_CreativeCommons_CopperTop_Type2_Small, Symbols:Symbol_CreativeCommons_CopperTop_Type2_Small, F.Cu at (137.3, 134.4)
- added REF***: OSHW-Symbol_6.7x6mm_Copper, Symbols:OSHW-Symbol_6.7x6mm_Copper, F.Cu at (144.0, 134.1)
- Q1: value Q_NMOS_GDS -> Q_NMOS_GSD
- moved R11 0.51 mm to (139.7, 142.4)
- moved R8 0.51 mm to (139.7, 147.4)
Connections:
- MK3 pad 1: GND -> (no net)
- MK4 pad 1: GND -> (no net)
- Q1 pad 2: Net-(Q1-Pad2) -> GNDD
- Q1 pad 3: GNDD -> Net-(Q1-Pad3)
- R3 pad 2: Net-(Q1-Pad2) -> Net-(Q1-Pad3)
- R4 pad 2: Net-(Q1-Pad2) -> Net-(Q1-Pad3)
Routing:
- net Net-(Q1-Pad2): track 12.0 -> 0.00 mm
- net Net-(Q1-Pad3): track 0.00 -> 11.4 mm
- net GNDD: track 11.3 -> 9.71 mm
- net VCC: track 87.5 -> 86.8 mm
- net Net-(R6-Pad1): track 43.1 -> 42.5 mm
Other:
- board text added: "2017-04.04"
